Commit message: Successful config for gazebo

File: urdf/leg.xacro (robot description, xacro)
@@ -1,23 +1,15 @@
-<?xml version="1.0"?>
 <robot name="noodle_leg" xmlns:xacro="http://www.ros.org/wiki/xacro">
-  <xacro:macro name="generic_cube_inertia" params="width height depth mass">
-    <inertial>
-      <mass value="${mass}"/>
-      <inertia ixx="${(mass/12.0) * (height**2 + depth**2)}" ixy="0.0" ixz="0.0"
-               iyy="${(mass/12.0) * (width**2 + depth**2)}" iyz="0.0"
-               izz="${(mass/12.0) * (width**2 + height**2)}"/>
-    </inertial>
-  </xacro:macro>
-  <xacro:property name="femur_w" value="0.01"/>
-  <xacro:property name="femur_l" value="0.01"/>
-  <xacro:property name="femur_h" value="0.3"/>
-  <xacro:property name="femur_w" value="0.01"/>
+  <link name="world"/>
+  <joint name="fixed" type="fixed">
+    <parent link="world"/>
+    <child link="femur"/>
+  </joint>
   <link name="femur">
     <visual>
       <geometry>
-        <box size="">
+        <mesh filename="package://noodle/cad/stl/femur.stl" scale="1e-3 1e-3 1e-3"/>
       </geometry>
     </visual>
+    <xacro:include filename="$(find noodle)/cad/urdf/femur.urdf"/>
   </link>
 </robot>
-</xml>

Commit message: adding models to urdf

File: urdf/leg.xacro (robot description, xacro)
@@ -1,6 +1,6 @@
 <robot name="noodle_leg" xmlns:xacro="http://www.ros.org/wiki/xacro">
-  <link name="world"/>
+  <link name="map"/>
   <joint name="fixed" type="fixed">
-    <parent link="world"/>
+    <parent link="map"/>
     <child link="femur"/>
   </joint>
@@ -13,3 +13,16 @@
     <xacro:include filename="$(find noodle)/cad/urdf/femur.urdf"/>
   </link>
+  <link name="servo">
+    <visual>
+      <geometry>
+        <mesh filename="package://noodle/cad/stl/servo.stl" scale="1e-3 1e-3 1e-3"/>
+      </geometry>
+    </visual>
+    <xacro:include filename="$(find noodle)/cad/urdf/servo.urdf"/>
+  </link>
+  <joint name="femur-to-servo" type="fixed">
+    <parent link="femur"/>
+    <child link="servo"/>
+    <origin xyz="24.2e-3 25e-3 250e-3" rpy="${pi/2} ${pi} 0"/>
+  </joint>
 </robot>
